File: lumberjack.kicad_pcb (KiCad board)
At the start: 2 copper layers, 284.7 x 94.2 mm, 165 parts, among them J1 USB, J2 AVR_ISP_6, J3 JST, J4 JST, J5 Molex, SW1 RESET, SW2 BOOT, U1 ATMEGA328-PU, Y1 16MHz

Commit message: Add hotswap MX design, attribution, and verified build documentation
Parts:
- removed 2u_MX30, 2u_MX60: SW_Push, lumberjack:MX_PCB_200B
- removed the REF** at (59.9, 73.2)
- MX1, MX10, MX11, MX12, MX13, MX14, MX15, MX16, MX17, MX18, MX19, MX2, MX20, MX21, MX22, MX23, MX24, MX25, MX26, MX27, MX28, MX29, MX3, MX30, MX31, MX32, MX33, MX34, MX35, MX36, MX37, MX38, MX39, MX4, MX40, MX41, MX42, MX43, MX44, MX45, MX46, MX47, MX48, MX49, MX5, MX50, MX51, MX52, MX53, MX54, MX55, MX56, MX57, MX58, MX59, MX6, MX60, MX7, MX9: footprint lumberjack:MX -> lumberjack_keyboard:CherryMX_Hotswap_1u
- MX8: footprint lumberjack:MX_NTHSTH -> lumberjack_keyboard:CherryMX_Hotswap_1u
- moved REF** 20.6 mm to (152.4, 100.3)
- moved REF** 2.38 mm to (240.5, 110.2)
- turned MX1 to 180 degrees
- turned MX7 to 180 degrees
Routing:
- net GND: track 75.3 -> 403.3 mm, vias 2 -> 32
- net /COL3: track 211.5 -> 168.4 mm, vias 1 -> 3
- net /COL1: track 239.9 -> 200.4 mm
- net /ROW1: track 101.2 -> 79.0 mm
- net /COL0: track 256.2 -> 234.1 mm, vias 0 -> 1
- net Net-(D60-A): track 35.5 -> 17.2 mm
- net Net-(D56-A): track 38.3 -> 20.1 mm
- net Net-(D55-A): track 46.8 -> 30.5 mm, vias 0 -> 1
- net Net-(D49-A): track 62.7 -> 47.4 mm, vias 0 -> 1
- net Net-(D3-A): track 108.8 -> 122.9 mm, vias 0 -> 1
- net Net-(D50-A): track 65.0 -> 50.9 mm, vias 0 -> 1
- net Net-(D4-A): track 110.2 -> 124.2 mm, vias 0 -> 1
- net Net-(D44-A): track 83.7 -> 69.9 mm, vias 0 -> 1
- net Net-(D47-A): track 62.6 -> 48.9 mm, vias 0 -> 1
- net Net-(D43-A): track 83.8 -> 70.4 mm, vias 0 -> 1
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